File: Schematics/RLS/RLS.kicad_pcb (KiCad board)
At the start: 2 copper layers, 1 part

Commit message: Removed duplicate folder
Removing duplicate folder Andrew created. Merged the schematic folder back where it should be for RLS.
Parts:
- removed P1: , 40pinRevised
- added C1, C2: 15pF, Capacitors_THT:C_Disc_D3.8mm_W2.6mm_P2.50mm, F.Cu at (135.9, 69.8)
- added C10, C12, C14, C22, C24, C26, C28, C30, C32, C39, C4, C40, C6, C8: 0.1uF, Capacitors_SMD:C_0603_HandSoldering, F.Cu at (135.9, 69.8)
- added C11, C13, C17, C18, C19, C20, C21, C23, C25, C27, C29, C3, C31, C35, C36, C37, C38, C41, C42, C45, C5, C7, C9: 10uF, Capacitors_SMD:CP_Elec_4x5.3, F.Cu at (135.9, 69.8)
- added C15, C16, C33, C34, C43, C44: 1uF, Capacitors_SMD:CP_Elec_4x5.3, F.Cu at (135.9, 69.8)
- added D1: AD_LED, LEDs:LED_0603, F.Cu at (135.9, 69.8)
- added D2: +5V_LED, LEDs:LED_0603, F.Cu at (135.9, 69.8)
- added DB1: BoardID_VIN_Scope_FuncGen_DB_CONN, Pin_Headers:Pin_Header_Straight_2x20_Pitch2.54mm, F.Cu at (152.4, 114.3)
- added DB2: Arduino_DB_CONN, Pin_Headers:Pin_Header_Straight_2x20_Pitch2.54mm, F.Cu at (182.9, 104.1)
- added DB3: Logic_Analyzer1_DB_CONN, Pin_Headers:Pin_Header_Straight_2x20_Pitch2.54mm, F.Cu at (254.0, 71.1)
- added DB4: Logic_Analyzer2_DB_CONN, Pin_Headers:Pin_Header_Straight_2x20_Pitch2.54mm, F.Cu at (168.9, 31.8)
- added F1: 1A, Fuse_Holders_and_Fuses:Fuse_SMD2920, F.Cu at (135.9, 69.8)
- added F2: 1.5A, Fuse_Holders_and_Fuses:Fuse_SMD2920, F.Cu at (135.9, 69.8)
- added F3: 4A, Fuse_Holders_and_Fuses:Fuse_SMD2920, F.Cu at (135.9, 69.8)
- added J1: Velleman_Probe1, Pin_Headers:Pin_Header_Straight_1x03_Pitch2.54mm, F.Cu at (135.9, 69.8)
- added J2: Velleman_Probe2, Pin_Headers:Pin_Header_Straight_1x03_Pitch2.54mm, F.Cu at (135.9, 69.8)
- added J3: Velleman_FuncGen, Pin_Headers:Pin_Header_Straight_1x03_Pitch2.54mm, F.Cu at (135.9, 69.8)
- added J4: Logic_Analyzer1, Pin_Headers:Pin_Header_Straight_2x20_Pitch2.54mm, F.Cu at (218.4, 68.6)
- added J5: Logic_Analyzer2, Pin_Headers:Pin_Header_Straight_2x20_Pitch2.54mm, F.Cu at (194.3, 29.2)
- added J6: ADS1115, Pin_Headers:Pin_Header_Straight_1x10_Pitch2.54mm, F.Cu at (64.8, 119.4)
- added J7: DC_Fan, Pin_Headers:Pin_Header_Straight_1x03_Pitch2.54mm, F.Cu at (135.9, 69.8)
- added PSU1: DIN_5, RLS_CustomFootprints:Molex_2x3_3.5mm, F.Cu at (135.9, 69.8)
- added Q1: BS170, TO_SOT_Packages_SMD:SOT-23, F.Cu at (135.9, 69.8)
- added R1, R10, R19, R2, R22, R3, R30, R31, R32, R33, R4, R5, R6, R7, R8, R9: 4.7K, Resistors_SMD:R_0805_HandSoldering, F.Cu at (135.9, 69.8)
- added R11, R13: 20K, Resistors_SMD:R_1206_HandSoldering, F.Cu at (135.9, 69.8)
- added R12, R14, R15, R16: 10K, Resistors_SMD:R_1206_HandSoldering, F.Cu at (135.9, 69.8)
- added R17, R18: 9M, Resistors_THT:R_Axial_DIN0309_L9.0mm_D3.2mm_P12.70mm_Horizontal, F.Cu at (135.9, 69.8)
- added R20, R21, R23, R24: 1.78K, Resistors_SMD:R_1206_HandSoldering, F.Cu at (135.9, 69.8)
- added R25, R28: 120, Resistors_SMD:R_1206_HandSoldering, F.Cu at (135.9, 69.8)
- added R26, R27: 1K_POT, Potentiometers:Potentiometer_Trimmer_Bourns_3296Y, F.Cu at (135.9, 69.8)
- added R29: 1K, Resistors_SMD:R_1206_HandSoldering, F.Cu at (135.9, 69.8)
- added TH1: 3K_NTC, Resistors_THT:R_Axial_DIN0411_L9.9mm_D3.6mm_P12.70mm_Horizontal, F.Cu at (135.9, 69.8)
- added U10, U11: LT1963, TO_SOT_Packages_THT:TO-220-5_Pentawatt_Multiwatt-5_Vertical_StaggeredType1, F.Cu at (135.9, 69.8)
- added U12: ULN2803A, Housings_DIP:DIP-18_W7.62mm, F.Cu at (38.1, 35.6)
- added U2: LM317T, TO_SOT_Packages_THT:TO-220_Vertical, F.Cu at (135.9, 69.8)
- added U3: LM337T, TO_SOT_Packages_THT:TO-220_Vertical, F.Cu at (135.9, 69.8)
- added U4, U5, U8, U9: AD5293, SMD_Packages:SSOP-14, F.Cu at (135.9, 69.8)
- added U6, U7: LT3015, TO_SOT_Packages_THT:TO-220-5_Pentawatt_Multiwatt-5_Vertical_StaggeredType1, F.Cu at (135.9, 69.8)
Other:
- board outline added: 228.6 x 228.6 mm
- copper layers 2 -> 4
- net class Default: clearance 0.2 -> 0.25
- rule trace_clearance: 0.2 -> 0.25
- rule trace_min: 0.2 -> 0.25

Commit message: CHANGE EVERYTHING
Parts:
- moved PSU1 139.2 mm to (36.8, 167.6)
- moved J3 131.4 mm to (25.4, 141.0)
- moved J7 124.8 mm to (34.3, 142.2)
- moved J1 122.7 mm to (27.9, 128.3)
- moved J2 116.7 mm to (35.6, 129.5)
- moved C44 92.6 mm to (54.6, 114.3)
- moved C43 89.2 mm to (54.6, 106.7)
- moved C31 88.2 mm to (54.6, 35.6)
- moved C42 86.4 mm to (54.6, 99.1)
- moved C33 85.2 mm to (54.6, 44.5)
- moved C41 83.2 mm to (55.9, 92.7)
- moved C34 83.2 mm to (54.6, 52.1)
- moved C38 82.7 mm to (54.6, 85.1)
- moved C45 82.1 mm to (66.0, 113.0)
- moved C35 81.9 mm to (54.6, 59.7)
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
Commit message: Lots of changes
Completed Schematic
1/3 Done PCB
Multisim file for testing ADC protection and buffer circuit
Parts:
- removed DB2: Arduino_DB_CONN, Pin_Headers:Pin_Header_Straight_2x20_Pitch2.54mm
- removed DB3: Logic_Analyzer1_DB_CONN, Pin_Headers:Pin_Header_Straight_2x20_Pitch2.54mm
- removed DB4: Logic_Analyzer2_DB_CONN, Pin_Headers:Pin_Header_Straight_2x20_Pitch2.54mm
- added R34: 10K, Resistors_SMD:R_1206_HandSoldering, F.Cu at (251.5, 40.6)
- added R35: 10K, Resistors_SMD:R_1206_HandSoldering, F.Cu at (251.5, 45.7)
- added R36: 10K, Resistors_SMD:R_1206_HandSoldering, F.Cu at (251.5, 50.8)
- added R37: 10K, Resistors_SMD:R_1206_HandSoldering, F.Cu at (251.5, 55.9)
- added R38: 1K, Resistors_SMD:R_1206_HandSoldering, F.Cu at (251.5, 61.0)
- added R39: 1K, Resistors_SMD:R_1206_HandSoldering, F.Cu at (251.5, 66.0)
- added U1: ARDUINO_MEGA_SHIELD, RLS_CustomFootprints:ARDUINO_MEGA_SHIELD, F.Cu at (125.1, 53.3)
- added U13: RA30421051, RLS_CustomFootprints:DIP-8(14)_W7.62mm, F.Cu at (83.8, 50.2)
- added U14: RA30421051, RLS_CustomFootprints:DIP-8(14)_W7.62mm, F.Cu at (83.8, 64.1)
- added U15: RB496EATR, TO_SOT_Packages_SMD:SOT-23-5_HandSoldering, F.Cu at (266.7, 63.5)
- added U16: RB496EATR, TO_SOT_Packages_SMD:SOT-23-5_HandSoldering, F.Cu at (266.7, 69.8)
- added U17: NE5532, Housings_SOIC:SOIC-8_3.9x4.9mm_Pitch1.27mm, F.Cu at (266.7, 77.5)
- added U18: NE5532, Housings_SOIC:SOIC-8_3.9x4.9mm_Pitch1.27mm, F.Cu at (266.7, 85.1)
- added U19: RB496EATR, TO_SOT_Packages_SMD:SOT-23-5_HandSoldering, F.Cu at (266.7, 92.7)
- added U20: RB496EATR, TO_SOT_Packages_SMD:SOT-23-5_HandSoldering, F.Cu at (266.7, 99.1)
- added U21: NE5532, Housings_SOIC:SOIC-8_3.9x4.9mm_Pitch1.27mm, F.Cu at (266.7, 106.7)
- DB1: value BoardID_VIN_Scope_FuncGen_DB_CONN -> DaughterBoard_Connectors; footprint Pin_Headers:Pin_Header_Straight_2x20_Pitch2.54mm -> RLS_CustomFootprints:Daughterboard_4_Conn
- R10, R8, R9: value 4.7K -> (none)
- R11: value 20K -> 120
- R12: value 10K -> 120
- R13: value 20K -> 1K
- R14: value 10K -> 1K
- R26, R27: footprint Potentiometers:Potentiometer_Trimmer_Bourns_3296Y -> Potentiometers:Potentiometer_Trimmer_Bourns_3266Y
- R3, R4, R5, R6, R7: value 4.7K -> ~
- moved J3 269.3 mm to (288.3, 199.4)
- moved C45 267.1 mm to (321.3, 34.3)
- moved J1 264.8 mm to (288.3, 176.5)
- moved C37 261.5 mm to (313.7, 41.9)
- moved C38 261.5 mm to (313.7, 49.5)
- moved C36 261.3 mm to (313.7, 34.3)
- moved J2 259.4 mm to (288.3, 188.0)
- moved J7 255.0 mm to (288.3, 165.1)
- moved C31 252.4 mm to (306.1, 57.1)
- moved C33 252.3 mm to (306.1, 64.8)
- moved C34 252.3 mm to (306.1, 72.4)
- moved C35 252.3 mm to (306.1, 80.0)
- moved C25 246.6 mm to (306.1, 34.3)
- moved C29 246.2 mm to (306.1, 49.5)
- moved C27 245.6 mm to (306.1, 41.9)
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Connections:
- net BID1 renamed /BID1
- net BID3 renamed /BID3
- net BID5 renamed /BID5
- net BID7 renamed /BID7
- net Net-(C1-Pad1) renamed /Scope_Probe_Gain/SCP1_10X
- net Net-(C15-Pad1) renamed /Negative_Regulators/-V1_EX_C
- net Net-(C16-Pad1) renamed /Negative_Regulators/-V2_EX_C
- net Net-(C33-Pad1) renamed /Positive_Regulators/+V1_EX_C
- net Net-(C34-Pad1) renamed /Positive_Regulators/+V2_EX_C
- net Net-(C41-Pad1) renamed /+5V_-5V_Regulators/+ADJ
- net Net-(C42-Pad2) renamed /+5V_-5V_Regulators/-ADJ
- net Net-(C45-Pad2) renamed /ADC_Divder_&_DC_Fan/FAN_GND
- net Net-(F1-Pad2) renamed /DIN-15
- net Net-(F2-Pad2) renamed /DIN+15
- net Net-(F3-Pad2) renamed /DIN5
- net Net-(Q1-Pad2) renamed /ADC_Divder_&_DC_Fan/VGS_FAN
- net Net-(R19-Pad1) renamed /Negative_Regulators/-SDO_SDI
- net Net-(R20-Pad1) renamed /Negative_Regulators/-V2_ADJ
- net Net-(R21-Pad1) renamed /Negative_Regulators/-V1_ADJ
- net Net-(R22-Pad1) renamed /Positive_Regulators/+SDO_SDI
- net Net-(R23-Pad1) renamed /Positive_Regulators/+V1_ADJ
- C2 pad 1: Net-(C2-Pad1) -> POS_SCP2
- C2 pad 2: POS_SCP2 -> /Scope_Probe_Gain/SCP2_10X
- DB1 pad 1: (no net) -> AA15
- DB1 pad 2: (no net) -> AA14
- DB1 pad 3: BID0 -> /BID0
- DB1 pad 5: BID2 -> /BID2
- DB1 pad 7: BID4 -> /BID4
- DB1 pad 9: BID6 -> /BID6
- J1 pad 2: (no net) -> Net-(J1-Pad2)
- J1 pad 3: (no net) -> /Scope_Probe_Gain/+SCP1
- J2 pad 2: (no net) -> Net-(J2-Pad2)
- J2 pad 3: (no net) -> /Scope_Probe_Gain/+SCP2
- J3 pad 2: (no net) -> Net-(J3-Pad2)
- J6 pad 10: VD03 -> AIN3
- J6 pad 3: (no net) -> SCL
- J6 pad 4: (no net) -> SDA
- J6 pad 6: (no net) -> Net-(J6-Pad6)
- J6 pad 7: VM00 -> AIN0
- J6 pad 8: VD01 -> AIN1
- J6 pad 9: VD02 -> AIN2
- J7 pad 3: (no net) -> Net-(J7-Pad3)
- R11 pad 1: VM03 -> /ADC_Divder_&_DC_Fan/-5_OVP
- R11 pad 2: VD03 -> VM02
- R12 pad 1: VD03 -> /ADC_Divder_&_DC_Fan/+5_OVP
- R12 pad 2: AGND -> VM00
- R13 pad 1: VM02 -> /ADC_Divder_&_DC_Fan/-5_INV
- R13 pad 2: VD02 -> /ADC_Divder_&_DC_Fan/-5_BUFF
- R14 pad 1: VD02 -> AIN2
- R14 pad 2: AGND -> /ADC_Divder_&_DC_Fan/-5_INV
- R15 pad 1: VM01 -> /ADC_Divder_&_DC_Fan/+15_OVP
- R15 pad 2: VD01 -> VM01
- R16 pad 1: VD01 -> /ADC_Divder_&_DC_Fan/+15_DIV
- R16 pad 2: AGND -> /ADC_Divder_&_DC_Fan/+15_OVP
- R18 pad 1: POS_SCP2 -> /Scope_Probe_Gain/SCP2_10X
- R18 pad 2: Net-(C2-Pad1) -> POS_SCP2
- R24 pad 1: Net-(R24-Pad1) -> /Positive_Regulators/+V2_ADJ
- R26 pad 1: (no net) -> Net-(R26-Pad1)
- R27 pad 3: (no net) -> Net-(R27-Pad3)
- R3 pad 1: BID6 -> /BID0
- R32 pad 1: (no net) -> AD_LED
- R4 pad 1: BID4 -> /BID2
- R5 pad 1: BID2 -> /BID4
- R6 pad 1: BID0 -> /BID6
- U10 pad 1: Net-(R24-Pad1) -> +V2_SHDN
- U10 pad 2: +V2 -> +15V
- U10 pad 4: +15V -> +V2
- U10 pad 5: (no net) -> /Positive_Regulators/+V2_ADJ
- U11 pad 1: (no net) -> +V1_SHDN
- U12 pad 11: (no net) -> Net-(U12-Pad11)
- U12 pad 12: (no net) -> Net-(U12-Pad12)
- U12 pad 13: (no net) -> Net-(U12-Pad13)
- U12 pad 14: (no net) -> Net-(U12-Pad14)
- U12 pad 15: (no net) -> Net-(U12-Pad15)
- U12 pad 16: (no net) -> Net-(U12-Pad16)
- U12 pad 17: (no net) -> RLY2
- U12 pad 18: (no net) -> RLY1
- U12 pad 3: (no net) -> Net-(U12-Pad3)
- U12 pad 4: (no net) -> Net-(U12-Pad4)
- U12 pad 5: (no net) -> Net-(U12-Pad5)
- U12 pad 6: (no net) -> Net-(U12-Pad6)
- U12 pad 7: (no net) -> Net-(U12-Pad7)
- U12 pad 8: (no net) -> Net-(U12-Pad8)
- U4 pad 14: (no net) -> Net-(U4-Pad14)
- U4 pad 3: (no net) -> Net-(U4-Pad3)
- U5 pad 13: (no net) -> Net-(U5-Pad13)
- U5 pad 14: (no net) -> Net-(U5-Pad14)
- U5 pad 3: (no net) -> Net-(U5-Pad3)
- U6 pad 1: (no net) -> -V2_SHDN
- U7 pad 1: (no net) -> -V1_SHDN
- U8 pad 14: (no net) -> Net-(U8-Pad14)
- U8 pad 3: (no net) -> Net-(U8-Pad3)
- U8 pad 4: Net-(R24-Pad1) -> /Positive_Regulators/+V2_ADJ
- U9 pad 13: (no net) -> Net-(U9-Pad13)
- U9 pad 14: (no net) -> Net-(U9-Pad14)
- U9 pad 3: (no net) -> Net-(U9-Pad3)
Routing:
- net +5V: track 0.00 -> 85.6 mm
- net POS_SCP1: track 0.00 -> 70.9 mm
- net POS_SCP2: track 0.00 -> 62.2 mm
- net AGND: track 0.00 -> 57.1 mm
- net -5V_R: track 0.00 -> 26.9 mm
- net /+5V_-5V_Regulators/-ADJ: track 0.00 -> 25.7 mm
- net +5V_R: track 0.00 -> 23.1 mm
- net RLY2: track 0.00 -> 21.2 mm
- net /Scope_Probe_Gain/SCP2_10X: track 0.00 -> 17.6 mm
- net /Scope_Probe_Gain/SCP1_10X: track 0.00 -> 17.6 mm
- net /BID7: track 0.00 -> 16.4 mm
- net /BID6: track 0.00 -> 16.4 mm
- net /BID5: track 0.00 -> 16.4 mm
- net /BID4: track 0.00 -> 16.4 mm
- net /BID3: track 0.00 -> 16.4 mm
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Other:
- board text added: "4.7K"

Commit message: Continued PCB and Final Schematic
Parts:
- C10, C12, C14, C22, C24, C26, C28, C30, C32, C39, C4, C40, C6, C8: footprint Capacitors_SMD:C_0603_HandSoldering -> Capacitors_SMD:C_1206_HandSoldering
- F1, F2, F3: footprint Fuse_Holders_and_Fuses:Fuse_SMD2920 -> RLS_CustomFootprints:Fuse_SMD_Custom
- R10, R8, R9: value (none) -> 4.7K
- R3, R4, R5, R6, R7: value ~ -> 4.7K
- moved J1 269.5 mm to (61.0, 31.8)
- moved J2 255.3 mm to (86.4, 31.8)
- moved R31 249.1 mm to (66.0, 191.8)
- moved J3 243.4 mm to (111.8, 31.8)
- moved R32 242.1 mm to (60.3, 179.1)
- moved D2 239.6 mm to (45.7, 191.1)
- moved D1 239.6 mm to (45.7, 187.3)
- moved R33 236.1 mm to (67.9, 184.2)
- moved R30 209.9 mm to (53.3, 189.9)
- moved F3 83.7 mm to (51.4, 206.4), turned to 270 degrees
- moved F2 74.6 mm to (62.9, 206.4), turned to 270 degrees
- moved F1 67.6 mm to (74.3, 206.4), turned to 270 degrees
- moved C41 27.1 mm to (99.1, 136.5)
- moved C43 27.1 mm to (108.0, 136.5)
- moved R27 27.1 mm to (85.1, 127.0)
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Connections:
- net Net-(D1-Pad1) renamed /ARD_LED
- net Net-(D2-Pad1) renamed /PSU_LED
- net Net-(R30-Pad1) renamed /ARD_R
- net Net-(R31-Pad1) renamed /PSU_R
Routing:
- net AA12: track 4.83 -> 92.7 mm
- net NEG_SCP1: track 0.00 -> 84.9 mm
- net AA13: track 11.0 -> 87.2 mm
- net L2GND: track 0.00 -> 74.9 mm
- net L1GND: track 0.00 -> 74.9 mm
- net NEG_SCP2: track 0.00 -> 65.3 mm
- net POS_SCP1: track 70.9 -> 124.4 mm
- net /BID0: track 16.4 -> 68.4 mm, vias 0 -> 2
- net NEG_GEN: track 0.00 -> 50.6 mm
- net /BID1: track 16.4 -> 66.8 mm, vias 0 -> 1
- net POS_GEN: track 0.00 -> 46.0 mm
- net POS_SCP2: track 62.2 -> 105.8 mm
- net /BID2: track 16.4 -> 59.7 mm, vias 0 -> 2
- net /BID3: track 16.4 -> 58.1 mm, vias 0 -> 1
- net /Scope_Probe_Gain/+SCP2: track 0.00 -> 38.8 mm
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
Commit message: PCB Layout 90% Done
All that is remaining is the LA traces (moved them and forgot to re-do them) and the SPI and SHDN lines for the digital pots and regs.
Also, do not merge this branch if you can. Have it fully replace the previous folder. There were obsolete files that I removed that Github keeps because it's dumb.
Parts:
- U10, U11, U6, U7: footprint TO_SOT_Packages_THT:TO-220-5_Pentawatt_Multiwatt-5_Vertical_StaggeredType1 -> RLS_CustomFootprints:TO-220-5_Vertical_Type1_w_Heatsink
- moved U5 265.8 mm to (78.7, 224.8), turned to 90 degrees
- moved C14 262.3 mm to (73.7, 217.8), turned to 180 degrees
- moved C11 262.1 mm to (88.3, 231.1), turned to 90 degrees
- moved C16 258.2 mm to (83.8, 177.8)
- moved C13 257.5 mm to (73.7, 210.8), turned to 180 degrees
- moved C19 257.1 mm to (109.2, 231.1), turned to 90 degrees
- moved C12 256.9 mm to (95.2, 231.1), turned to 270 degrees
- moved C5 255.8 mm to (88.3, 198.1), turned to 90 degrees
- moved C10 252.3 mm to (94.0, 217.8), turned to 180 degrees
- moved C7 252.2 mm to (73.7, 177.8), turned to 180 degrees
- moved C8 251.1 mm to (73.7, 184.8), turned to 180 degrees
- moved C9 249.7 mm to (94.0, 210.8), turned to 180 degrees
- moved U4 249.3 mm to (78.7, 191.8), turned to 90 degrees
- moved C17 245.4 mm to (109.2, 198.1), turned to 90 degrees
- moved C6 245.1 mm to (95.2, 198.1), turned to 270 degrees
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Routing:
- net -15V: track 13.3 -> 472.3 mm, vias 0 -> 10
- net +15V: track 11.8 -> 384.2 mm, vias 0 -> 9
- net +5V: track 53.9 -> 425.2 mm, vias 0 -> 7
- net AGND: track 65.5 -> 328.5 mm, vias 0 -> 9
- net +V2: track 0.00 -> 231.2 mm, vias 0 -> 3
- net -V1: track 0.00 -> 202.4 mm, vias 0 -> 3
- net +V1: track 0.00 -> 197.5 mm, vias 0 -> 2
- net -V2: track 0.00 -> 169.6 mm, vias 0 -> 4
- net -5V_R: track 43.8 -> 186.8 mm, vias 0 -> 3
- net SCLK: track 0.00 -> 141.8 mm, vias 0 -> 4
- net +5V_R: track 34.7 -> 167.6 mm, vias 0 -> 2
- net N_POT_CE: track 0.00 -> 101.9 mm
- net P_POT_CE: track 0.00 -> 100.4 mm
- net SDA: track 0.00 -> 98.8 mm, vias 0 -> 1
- net AIN0: track 0.00 -> 96.1 mm
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- added copper zone on Lower, net +15V
- added copper zone on Lower, net +5V
- added copper zone on F.Cu, net +5V_R
- added copper zone on Lower, net -15V
- added copper zone on F.Cu, net -5V_R
- added copper zone on Upper, net AGND
- added copper zone on B.Cu, net DGND
Other:
- board text added: "O"

Commit message: Finished PCB but...
Somehow managed to break the schematic file. I know how to fix it, but it is tedious and pointless for now (one has to go through every single individual component and verify that it is the same in the PCB, since the annotation script fucked everything up in the schematic, and therefore any new Netlist).
Parts:
- D1, D2, R30, R31, R32, R33: moved to B.Cu
- moved D2 306.2 mm to (247.0, 31.1)
- moved D1 303.4 mm to (247.0, 43.2)
- moved R30 286.9 mm to (237.5, 43.2)
- moved R31 277.2 mm to (237.5, 31.1)
- moved R32 269.5 mm to (228.6, 43.2)
- moved R33 265.0 mm to (228.6, 31.1)
- moved J7 250.8 mm to (46.4, 234.3), turned to 180 degrees
- moved C45 163.2 mm to (141.0, 211.5), turned to 0 degrees
- moved TH1 136.0 mm to (139.1, 201.3)
- moved Q1 129.5 mm to (156.2, 212.1)
- moved R29 121.4 mm to (156.2, 218.4)
Routing:
- net +5V: track 425.2 -> 794.4 mm
- net MOSI: track 83.3 -> 332.5 mm
- net L1GND: track 0.00 -> 248.7 mm
- net L2GND: track 0.00 -> 243.5 mm
- net SCLK: track 141.8 -> 376.8 mm, vias 4 -> 6
- net AD_LED: track 0.00 -> 171.5 mm
- net AGND: track 328.5 -> 499.0 mm, vias 9 -> 21
- net N_POT_CE: track 101.9 -> 243.4 mm, vias 0 -> 1
- net /ADC_Divder_&_DC_Fan/FAN_GND: track 0.00 -> 133.8 mm, vias 0 -> 2
- net +V2_SHDN: track 45.6 -> 175.6 mm, vias 0 -> 1
- net P_POT_CE: track 100.4 -> 220.8 mm, vias 0 -> 1
- net -15V: track 472.3 -> 588.3 mm, vias 10 -> 11
- net +V1_SHDN: track 43.6 -> 140.3 mm, vias 0 -> 1
- net -V1_SHDN: track 48.7 -> 140.1 mm, vias 0 -> 2
- net -V2_SHDN: track 51.7 -> 109.0 mm
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- added copper zone on Upper, net +15V
Other:
- board text added: "+5V Power"
- board text added: "Arduino Power"
