File: Schematics/RLS/RLS.kicad_pcb (KiCad board)
At the start: 4 copper layers, 200.7 x 215.9 mm, 127 parts, among them J1 ADS1115, J2 DC_Fan, J3 Velleman_Probe1, J4 Velleman_FuncGen, J5 Velleman_Probe2, J6 Logic_Analyzer1, J7 Logic_Analyzer2, Q1 BS170, U1 ARDUINO_MEGA_SHIELD, U10 RA30421051, U11 RA30421051, U12 AD5293, U13 AD5293, U14 LT3015, U15 LT3015, U16 AD5293, U17 AD5293, U18 LT1963, U19 LT1963, U2 RB496EATR, U20 LM317T, U21 LM337T, U3 RB496EATR, U4 NE5532, U5 NE5532, U6 RB496EATR, U7 RB496EATR, U8 NE5532, U9 ULN2803A

Commit message: Finished PCB Need to do Gerbers
It needs to be bought
Parts:
- removed the REF** at (115.6, 182.2)
- added REF**: MountingHole_3.5mm, Mounting_Holes:MountingHole_3.5mm, F.Cu at (111.8, 181.6)
- added REF**: MountingHole_3.5mm, Mounting_Holes:MountingHole_3.5mm, F.Cu at (25.4, 181.6)
- DB1: footprint RLS_CustomFootprints:Daughterboard_4_Conn -> Daughterboard_4_Conn
- F1: footprint RLS_CustomFootprints:Fuse_SMD_Custom -> Fuse_SMD_Custom
- PSU1: footprint RLS_CustomFootprints:Molex_2x3_3.5mm -> Molex_2x3_3.5mm
- RV1: footprint RLS_CustomFootprints:Potentiometer_Trimmer_Bourns_PVG5A -> Potentiometer_Trimmer_Bourns_PVG5A
- U1: footprint RLS_CustomFootprints:ARDUINO_MEGA_SHIELD -> ARDUINO_MEGA_SHIELD
- U15: footprint RLS_CustomFootprints:TO-220-5_Vertical_Type1_w_Heatsink -> TO-220-5_Vertical_Type1_w_Heatsink
- moved REF** 46.0 mm to (99.1, 131.4)
- moved REF** 22.6 mm to (185.4, 131.4)
- moved D1 17.2 mm to (186.1, 37.5)
- moved D2 17.2 mm to (186.1, 23.5)
- moved J6 10.8 mm to (151.1, 38.1)
- moved J7 10.8 mm to (172.7, 38.1)
- moved C3 8.35 mm to (85.1, 28.6), turned to 0 degrees
- moved C31 6.99 mm to (169.5, 172.1)
- moved C35 6.99 mm to (169.5, 205.1)
- moved C38 6.99 mm to (153.7, 192.4)
- moved C39 6.99 mm to (153.7, 225.4)
- moved R31 6.99 mm to (179.1, 205.7)
- moved U16 6.99 mm to (179.1, 178.4)
- moved U17 6.99 mm to (179.1, 211.5)
- moved U18 6.99 mm to (131.4, 194.3)
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Connections:
- D1 pad 1: /ARD_LED -> DGND
- D1 pad 2: AGND -> /ARD_LED
- D2 pad 1: /PSU_LED -> AGND
- D2 pad 2: AGND -> /PSU_LED
- J1 pad 6: (no net) -> Net-(J1-Pad6)
- J2 pad 3: (no net) -> Net-(J2-Pad3)
- J3 pad 2: (no net) -> Net-(J3-Pad2)
- J4 pad 2: (no net) -> Net-(J4-Pad2)
- J5 pad 2: (no net) -> Net-(J5-Pad2)
- RV1 pad 1: (no net) -> Net-(RV1-Pad1)
- RV2 pad 3: (no net) -> Net-(RV2-Pad3)
- RV3 pad 1: (no net) -> Net-(RV3-Pad1)
- RV4 pad 1: (no net) -> Net-(RV4-Pad1)
- RV5 pad 1: (no net) -> Net-(RV5-Pad1)
- U1 pad 0: (no net) -> Net-(U1-Pad0)
- U1 pad 1: (no net) -> Net-(U1-Pad1)
- U1 pad 14: (no net) -> Net-(U1-Pad14)
- U1 pad 15: (no net) -> Net-(U1-Pad15)
- U1 pad 16: (no net) -> Net-(U1-Pad16)
- U1 pad 17: (no net) -> Net-(U1-Pad17)
- U1 pad 18: (no net) -> Net-(U1-Pad18)
- U1 pad 19: (no net) -> Net-(U1-Pad19)
- U1 pad 2: (no net) -> Net-(U1-Pad2)
- U1 pad 3: (no net) -> Net-(U1-Pad3)
- U1 pad 3V3: (no net) -> Net-(U1-Pad3V3)
- U1 pad 4: (no net) -> Net-(U1-Pad4)
- U1 pad 49: (no net) -> Net-(U1-Pad49)
- U1 pad 5: (no net) -> Net-(U1-Pad5)
- U1 pad 5V_4: (no net) -> Net-(U1-Pad5V_4)
- U1 pad 5V_5: (no net) -> Net-(U1-Pad5V_5)
- U1 pad 6: (no net) -> Net-(U1-Pad6)
- U1 pad 7: (no net) -> Net-(U1-Pad7)
- U1 pad 8: (no net) -> Net-(U1-Pad8)
- U1 pad AREF: (no net) -> Net-(U1-PadAREF)
- U1 pad GND2: (no net) -> DGND
- U1 pad GND3: (no net) -> Net-(U1-PadGND3)
- U1 pad GND4: (no net) -> Net-(U1-PadGND4)
- U1 pad GND5: (no net) -> Net-(U1-PadGND5)
- U1 pad RST: (no net) -> Net-(U1-PadRST)
- U10 pad 5: (no net) -> Net-(U10-Pad5)
- U10 pad 6: (no net) -> Net-(U10-Pad6)
- U10 pad 7: (no net) -> Net-(U10-Pad7)
- U11 pad 5: (no net) -> Net-(U11-Pad5)
- U11 pad 6: (no net) -> Net-(U11-Pad6)
- U11 pad 7: (no net) -> Net-(U11-Pad7)
- U12 pad 13: (no net) -> Net-(U12-Pad13)
- U12 pad 14: (no net) -> Net-(U12-Pad14)
- U12 pad 3: (no net) -> Net-(U12-Pad3)
- U13 pad 14: (no net) -> Net-(U13-Pad14)
- U13 pad 3: (no net) -> Net-(U13-Pad3)
- U16 pad 13: (no net) -> Net-(U16-Pad13)
- U16 pad 14: (no net) -> Net-(U16-Pad14)
- U16 pad 3: (no net) -> Net-(U16-Pad3)
- U17 pad 14: (no net) -> Net-(U17-Pad14)
- U17 pad 3: (no net) -> Net-(U17-Pad3)
- U2 pad 2: (no net) -> Net-(U2-Pad2)
- U3 pad 2: (no net) -> Net-(U3-Pad2)
- U6 pad 2: (no net) -> Net-(U6-Pad2)
- U7 pad 2: (no net) -> Net-(U7-Pad2)
- U9 pad 11: (no net) -> Net-(U9-Pad11)
- U9 pad 12: (no net) -> Net-(U9-Pad12)
- U9 pad 13: (no net) -> Net-(U9-Pad13)
- U9 pad 14: (no net) -> Net-(U9-Pad14)
- U9 pad 15: (no net) -> Net-(U9-Pad15)
- U9 pad 16: (no net) -> Net-(U9-Pad16)
- U9 pad 3: (no net) -> Net-(U9-Pad3)
- U9 pad 4: (no net) -> Net-(U9-Pad4)
- U9 pad 5: (no net) -> Net-(U9-Pad5)
- U9 pad 6: (no net) -> Net-(U9-Pad6)
- U9 pad 7: (no net) -> Net-(U9-Pad7)
- U9 pad 8: (no net) -> Net-(U9-Pad8)
Routing:
- net DGND: track 0.00 -> 188.7 mm
- net L2GND: track 250.7 -> 201.2 mm
- net L1GND: track 250.7 -> 201.2 mm
- net AD_LED: track 171.2 -> 198.3 mm
- net AGND: track 509.8 -> 482.6 mm
- net +5V_R: track 203.1 -> 177.2 mm
- net -15V: track 595.3 -> 576.7 mm
- net +5V: track 728.4 -> 744.9 mm, vias 7 -> 8
- net L2CLK2: track 47.3 -> 34.3 mm
- net L1CLK2: track 47.3 -> 34.3 mm
- net L2D30: track 41.1 -> 32.2 mm
- net L1D30: track 41.1 -> 32.2 mm
- net L2D24: track 40.8 -> 32.6 mm
- net L2D18: track 40.8 -> 32.6 mm
- net L1D24: track 40.8 -> 32.6 mm
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- added copper zone on F.Cu, net +5V_R
- added copper zone on F.Cu, net -15V
Other:
- board text added: "Designed by: Andrew Soshea Gregory Asher Gytautas Jankauskas Paolo Sebastian"
- board text added: "REMOTE LAB SYSTEM"
- board text added: "UWB"

Commit message: Made a few minor changes...
To the PCB. Also added the gerber files and fixed/added objects for the 3D visualization
Parts:
- J6: footprint Pin_Headers:Pin_Header_Straight_2x20_Pitch2.54mm -> Pin_Header_Straight_2x20_Pitch2.54mm
- RV1: footprint Potentiometer_Trimmer_Bourns_PVG5A -> RLS_CustomFootprints:Potentiometer_Trimmer_Bourns_PVG5A
- U15: footprint TO-220-5_Vertical_Type1_w_Heatsink -> RLS_CustomFootprints:TO-220-5_Vertical_Type1_w_Heatsink
- moved REF** 7.73 mm to (193.0, 132.7)
- moved REF** 7.73 mm to (106.7, 132.7)
- moved C13 7.62 mm to (62.9, 224.2)
- moved C17 7.62 mm to (62.9, 191.1)
- moved C22 7.62 mm to (181.6, 192.4)
- moved C23 7.62 mm to (181.6, 225.4)
- moved C24 7.62 mm to (191.8, 192.4)
- moved C25 7.62 mm to (191.8, 185.4)
- moved C26 7.62 mm to (191.8, 225.4)
- moved C27 7.62 mm to (191.8, 218.4)
- moved C30 7.62 mm to (170.2, 172.1)
- moved C31 7.62 mm to (177.2, 172.1)
- moved C34 7.62 mm to (170.2, 205.1)
- moved C35 7.62 mm to (177.2, 205.1)
- moved C36 7.62 mm to (156.2, 172.1)
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Other:
- board text added: "UWB REMOTE LAB SYSTEM"
- board text removed: "REMOTE LAB SYSTEM"
- board text removed: "UWB"
