File: Schematics/RLS/RLS.sch (KiCad schematic (older format))
At the start: 24 parts, among them J6 ADS1115, U1 ARDUINO_MEGA_SHIELD

Commit message: Lots of changes
Completed Schematic
1/3 Done PCB
Multisim file for testing ADC protection and buffer circuit
Parts:
- removed DB1: BoardID_VIN_Scope_FuncGen_DB_CONN, Pin_Headers:Pin_Header_Straight_2x20_Pitch2.54mm, symbol CONN_02X20
- removed DB2: Arduino_DB_CONN, Pin_Headers:Pin_Header_Straight_2x20_Pitch2.54mm, symbol CONN_02X20
- removed DB3: Logic_Analyzer1_DB_CONN, Pin_Headers:Pin_Header_Straight_2x20_Pitch2.54mm, symbol CONN_02X20
- removed DB4: Logic_Analyzer2_DB_CONN, Pin_Headers:Pin_Header_Straight_2x20_Pitch2.54mm, symbol CONN_02X20
- added DB1: DaughterBoard_Connectors, RLS_CustomFootprints:Daughterboard_4_Conn, symbol DaughterBoard_Connectors
- U1: footprint (none) -> RLS_CustomFootprints:ARDUINO_MEGA_SHIELD
Connections:
- net +15V: now also DB1.25 (+15V), DB1.27 (+15V)
- net +5V_R: now also DB1.33 (+5V_Reg), DB1.35 (+5V_Reg)
- net +V1: now also DB1.17 (+V1)
- net +V2: now also DB1.19 (+V2)
- net -15V: now also DB1.29 (-15V), DB1.31 (-15V)
- net -5V_R: now also DB1.37 (-5V_Reg), DB1.39 (-5V_Reg)
- net -V1: now also DB1.21 (-V1)
- net -V2: now also DB1.23 (-V2)
- net AA14: now also DB1.2 (AA14)
- net AA15: now also DB1.1 (AA15)
- net AD10: now also DB1.54 (AD10)
- net AD11: now also DB1.56 (AD11)
- net AD12: now also DB1.58 (AD12)
- net AD13: now also DB1.60 (AD13)
- net AD22: now also DB1.62 (AD22)
- net AD23: now also DB1.64 (AD23)
- net AD24: now also DB1.66 (AD24)
- net AD25: now also DB1.68 (AD25)
- net AD26: now also DB1.70 (AD26)
- net AD27: now also DB1.72 (AD27)
- net AD28: now also DB1.74 (AD28)
- net AD29: now also DB1.76 (AD29)
- net AD30: now also DB1.78 (AD30)
- net AD31: now also DB1.80 (AD31)
- net AD32: now also DB1.41 (AD32)
- net AD33: now also DB1.43 (AD33)
- net AD34: now also DB1.45 (AD34)
- net AD35: now also DB1.47 (AD35)
- net AD36: now also DB1.49 (AD36)
- net AD37: now also DB1.51 (AD37)
- net AD38: now also DB1.53 (AD38)
- net AD39: now also DB1.55 (AD39)
- net AD4: now also DB1.42 (AD4)
- net AD40: now also DB1.57 (AD40)
- net AD41: now also DB1.59 (AD41)
- net AD42: now also DB1.61 (AD42)
- net AD43: now also DB1.63 (AD43)
- net AD44: now also DB1.65 (AD44)
- net AD45: now also DB1.67 (AD45)
- net AD46: now also DB1.69 (AD46)
- net AD47: now also DB1.71 (AD47)
- net AD5: now also DB1.44 (AD5)
- net AD6: now also DB1.46 (AD6)
- net AD7: now also DB1.48 (AD7)
- net AD8: now also DB1.50 (AD8)
- net AD9: now also DB1.52 (AD9)
- net AGND: now also DB1.30 (AGND), DB1.32 (AGND), DB1.34 (AGND), DB1.36 (AGND), DB1.38 (AGND), DB1.40 (AGND)
- net BID0: now also R3.1, DB1.3 (BID0); no longer R6.1
- net BID1: now also DB1.4 (BID1)
- net BID2: now also R4.1, DB1.5 (BID2); no longer R5.1
- net BID3: now also DB1.6 (BID3)
- net BID4: now also R5.1, DB1.7 (BID4); no longer R4.1
- net BID5: now also DB1.8 (BID5)
- net BID6: now also R6.1, DB1.9 (BID6); no longer R3.1
- net BID7: now also DB1.10 (BID7)
- net DGND: now also DB1.18 (DGND), DB1.20 (DGND), DB1.22 (DGND), DB1.24 (DGND), DB1.26 (DGND), DB1.28 (DGND)
- net L1CLK1: now also DB1.100 (L1CLK1)
- net L1CLK2: now also DB1.120 (L1CLK2)
- net L1D0: now also DB1.81 (L1D0)
- net L1D1: now also DB1.82 (L1D1)
- net L1D10: now also DB1.93 (L1D10)
- net L1D11: now also DB1.94 (L1D11)
- net L1D12: now also DB1.95 (L1D12)
- net L1D13: now also DB1.96 (L1D13)
- net L1D14: now also DB1.97 (L1D14)
- net L1D15: now also DB1.98 (L1D15)
- net L1D16: now also DB1.101 (L1D16)
- net L1D17: now also DB1.102 (L1D17)
- net L1D18: now also DB1.103 (L1D18)
- net L1D19: now also DB1.104 (L1D19)
- net L1D2: now also DB1.83 (L1D2)
- net L1D20: now also DB1.105 (L1D20)
- net L1D21: now also DB1.106 (L1D21)
- net L1D22: now also DB1.107 (L1D22)
- net L1D23: now also DB1.108 (L1D23)
- net L1D24: now also DB1.111 (L1D24)
- net L1D25: now also DB1.112 (L1D25)
- net L1D26: now also DB1.113 (L1D26)
- net L1D27: now also DB1.114 (L1D27)
- net L1D28: now also DB1.115 (L1D28)
- net L1D29: now also DB1.116 (L1D29)
- net L1D3: now also DB1.84 (L1D3)
- net L1D30: now also DB1.117 (L1D30)
- net L1D31: now also DB1.118 (L1D31)
- net L1D4: now also DB1.85 (L1D4)
- net L1D5: now also DB1.86 (L1D5)
- net L1D6: now also DB1.87 (L1D6)
- net L1D7: now also DB1.88 (L1D7)
- net L1D8: now also DB1.91 (L1D8)
- net L1D9: now also DB1.92 (L1D9)
- net L1GND: now also DB1.109 (L1GND), DB1.110 (L1GND), DB1.119 (L1GND), DB1.89 (L1GND), DB1.90 (L1GND), DB1.99 (L1GND)
- net L2CLK1: now also DB1.140 (L2CLK1)
- net L2CLK2: now also DB1.160 (L2CLK2)
- net L2D0: now also DB1.121 (L2D0)
- net L2D1: now also DB1.122 (L2D1)
- net L2D10: now also DB1.133 (L2D10)
- net L2D11: now also DB1.134 (L2D11)
- net L2D12: now also DB1.135 (L2D12)
- net L2D13: now also DB1.136 (L2D13)
- net L2D14: now also DB1.137 (L2D14)
- net L2D15: now also DB1.138 (L2D15)
- net L2D16: now also DB1.141 (L2D16)
- net L2D17: now also DB1.142 (L2D17)
- net L2D18: now also DB1.143 (L2D18)
- net L2D19: now also DB1.144 (L2D19)
- net L2D2: now also DB1.123 (L2D2)
- net L2D20: now also DB1.145 (L2D20)
- net L2D21: now also DB1.146 (L2D21)
- net L2D22: now also DB1.147 (L2D22)
- net L2D23: now also DB1.148 (L2D23)
- net L2D24: now also DB1.151 (L2D24)
- net L2D25: now also DB1.152 (L2D25)
- net L2D26: now also DB1.153 (L2D26)
- net L2D27: now also DB1.154 (L2D27)
- net L2D28: now also DB1.155 (L2D28)
- net L2D29: now also DB1.156 (L2D29)
- net L2D3: now also DB1.124 (L2D3)
- net L2D30: now also DB1.157 (L2D30)
- net L2D31: now also DB1.158 (L2D31)
- net L2D4: now also DB1.125 (L2D4)
- net L2D5: now also DB1.126 (L2D5)
- net L2D6: now also DB1.127 (L2D6)
- net L2D7: now also DB1.128 (L2D7)
- net L2D8: now also DB1.131 (L2D8)
- net L2D9: now also DB1.132 (L2D9)
- net L2GND: now also DB1.129 (L2GND), DB1.130 (L2GND), DB1.139 (L2GND), DB1.149 (L2GND), DB1.150 (L2GND), DB1.159 (L2GND)
- net NEG_GEN: now also DB1.12 (-FG)
- net NEG_SCP1: now also DB1.14 (-SPC1)
- net NEG_SCP2: now also DB1.16 (-SPC2)
- net POS_GEN: now also DB1.11 (+FG)
- net POS_SCP1: now also DB1.13 (+SCP1)
- net POS_SCP2: now also DB1.15 (+SCP2)
- net VM00: now also DB1.73 (VM00); no longer J6.7 (P7)
- net VM01: now also DB1.75 (VM01)
- net VM02: now also DB1.77 (VM02)
- net VM03: now also DB1.79 (VM03)
- net DIN5: now reaches F3.2, PSU1.3
- net DIN-15: now reaches F1.2, PSU1.4
- net DIN+15: now reaches F2.2, PSU1.5
- net VD01 renamed AIN1
- net VD02 renamed AIN2
- net VD03 renamed AIN3
- new net AIN0: J6.7 (P7)
Other:
- note added: "VOLTMETER NOTES:\nVM00 MAX: + 5V\nVM01 MAX: + 15V\nVM02 MAX: - 5V\nVM03 MAX: - 15V"
- note removed: "VOLTMETER NOTES:\nVM00 MAX RANGE +/- 5V\nVM01 MAX RANGE +/- 10V\nVM02 MAX RANGE +/- 15V\nVM03 MAX RANGE +/- 15V"
- moved on the sheet: R10, R3, R4, R5, R6, R7, R8, R9, U1

Commit message: Continued PCB and Final Schematic
Parts:
- F1, F2, F3: footprint Fuse_Holders_and_Fuses:Fuse_SMD2920 -> RLS_CustomFootprints:Fuse_SMD_Custom
Connections:
- net ARD_LED: now reaches D1.1 (K), R30.2
- net PSU_LED: now reaches D2.1 (K), R31.2
- net ARD_R: now reaches R30.1, R32.2
- net PSU_R: now reaches R31.1, R33.2
Changed lines of the file:
@@
 F 0 "F3" H 2450 690 50  0000 C CNN
 F 1 "4A" H 2450 810 50  0000 C CNN
-F 2 "Fuse_Holders_and_Fuses:Fuse_SMD2920" H 2450 750 50  0001 C CNN
+F 2 "RLS_CustomFootprints:Fuse_SMD_Custom" H 2450 750 50  0001 C CNN
 F 3 "" H 2450 750 50  0001 C CNN
 	1    2450 750
@@
 F 0 "F2" H 1950 690 50  0000 C CNN
 F 1 "1.5A" H 1950 810 50  0000 C CNN
-F 2 "Fuse_Holders_and_Fuses:Fuse_SMD2920" H 1950 750 50  0001 C CNN
+F 2 "RLS_CustomFootprints:Fuse_SMD_Custom" H 1950 750 50  0001 C CNN
 F 3 "" H 1950 750 50  0001 C CNN
 	1    1950 750
@@
 F 0 "F1" H 1150 1190 50  0000 C CNN
 F 1 "1A" H 1150 1310 50  0000 C CNN
-F 2 "Fuse_Holders_and_Fuses:Fuse_SMD2920" H 1150 1250 50  0001 C CNN
+F 2 "RLS_CustomFootprints:Fuse_SMD_Custom" H 1150 1250 50  0001 C CNN
 F 3 "" H 1150 1250 50  0001 C CNN
 	1    1150 1250
@@
 Text Label 1300 1250 1    60   ~ 0
 DIN-15
+Text Label 1200 4750 2    60   ~ 0
+ARD_LED
+Text Label 1650 4750 0    60   ~ 0
+PSU_LED
+Text Label 1200 4300 2    60   ~ 0
+ARD_R
+Text Label 1650 4300 0    60   ~ 0
+PSU_R
 $EndSCHEMATC

Commit message: Finished PCB but...
Somehow managed to break the schematic file. I know how to fix it, but it is tedious and pointless for now (one has to go through every single individual component and verify that it is the same in the PCB, since the annotation script fucked everything up in the schematic, and therefore any new Netlist).
Changed lines of the file:
@@
 +5V_LED
-$Comp
-L R R32
-U 1 1 595DF587
-P 1200 4100
-F 0 "R32" V 1280 4100 50  0000 C CNN
-F 1 "4.7K" V 1200 4100 50  0000 C CNN
-F 2 "Resistors_SMD:R_0805_HandSoldering" V 1130 4100 50  0001 C CNN
-F 3 "" H 1200 4100 50  0001 C CNN
-	1    1200 4100
-	1    0    0    -1
-$EndComp
-$Comp
-L R R33
-U 1 1 595DF58E
-P 1650 4100
-F 0 "R33" V 1730 4100 50  0000 C CNN
-F 1 "4.7K" V 1650 4100 50  0000 C CNN
-F 2 "Resistors_SMD:R_0805_HandSoldering" V 1580 4100 50  0001 C CNN
-F 3 "" H 1650 4100 50  0001 C CNN
-	1    1650 4100
-	1    0    0    -1
-$EndComp
 $Comp
 L ARDUINO_MEGA_SHIELD U1
@@
 	2150 750  2050 750
 Wire Wire Line
-	850  1250 1050 1250
-Wire Wire Line
-	1350 750  1850 750
+	850  1250 950  1250
+Wire Wire Line
+	950  1250 1050 1250
+Wire Wire Line
+	1350 750  1600 750
+Wire Wire Line
+	1600 750  1850 750
 Wire Wire Line
 	1350 1250 1250 1250
@@
 	1500 2300 1850 2300
 Wire Wire Line
-	1850 2300 1850 2600
+	1850 2300 1850 2450
+Wire Wire Line
+	1850 2450 1850 2600
 Wire Wire Line
 	1850 2600 1500 2600
@@
 Connection ~ 1850 2450
 Wire Wire Line
-	10975 2575 11100 2575
-Wire Wire Line
-	11025 2575 11025 3125
+	10975 2575 11025 2575
+Wire Wire Line
+	11025 2575 11100 2575
+Wire Wire Line
+	11025 2575 11025 2750
+Wire Wire Line
+	11025 2750 11025 2950
+Wire Wire Line
+	11025 2950 11025 3125
 Wire Wire Line
 	11025 3125 10975 3125
@@
 	9325 1525 9325 975
 Wire Wire Line
-	1700 950  1950 950
+	1700 950  1750 950
+Wire Wire Line
+	1750 950  1950 950
 Wire Wire Line
 	1750 950  1750 1050
 Wire Wire Line
-	1000 1450 1350 1450
+	1000 1450 1250 1450
+Wire Wire Line
+	1250 1450 1350 1450
 Wire Wire Line
 	1250 1450 1250 1600
@@
 Connection ~ 1750 950
 Wire Wire Line
-	10100 4050 10100 4550
-Wire Wire Line
-	10050 4550 10150 4550
+	10100 4050 10100 4150
+Wire Wire Line
+	10100 4150 10100 4250
+Wire Wire Line
+	10100 4250 10100 4350
+Wire Wire Line
+	10100 4350 10100 4450
+Wire Wire Line
+	10100 4450 10100 4550
+Wire Wire Line
+	10050 4550 10100 4550
+Wire Wire Line
+	10100 4550 10150 4550
 Wire Wire Line
 	10050 4450 10100 4450
@@
 	10050 3450 10100 3450
 Wire Wire Line
-	10100 3450 10100 3950
-Wire Wire Line
-	10050 3950 10150 3950
+	10100 3450 10100 3550
+Wire Wire Line
+	10100 3550 10100 3650
+Wire Wire Line
+	10100 3650 10100 3750
+Wire Wire Line
+	10100 3750 10100 3850
+Wire Wire Line
+	10100 3850 10100 3950
+Wire Wire Line
+	10050 3950 10100 3950
+Wire Wire Line
+	10100 3950 10150 3950
 Wire Wire Line
 	10050 3850 10100 3850
@@
 	2250 750  2250 1450
 Wire Wire Line
-	2550 750  2800 750
+	2550 750  2650 750
+Wire Wire Line
+	2650 750  2800 750
 Connection ~ 2650 750
 Wire Wire Line
 	1650 5200 1650 5150
 Wire Wire Line
-	1200 5200 1650 5200
+	1200 5200 1400 5200
+Wire Wire Line
+	1400 5200 1650 5200
 Wire Wire Line
 	1200 5200 1200 5150
@@
 	10575 3125 10675 3125
 Wire Wire Line
-	7950 2575 8125 2575
-Wire Wire Line
-	8025 2575 8025 3125
+	7950 2575 8025 2575
+Wire Wire Line
+	8025 2575 8125 2575
+Wire Wire Line
+	8025 2575 8025 2750
+Wire Wire Line
+	8025 2750 8025 2950
+Wire Wire Line
+	8025 2950 8025 3125
 Wire Wire Line
 	8025 3125 8125 3125
@@
 Text Label 1650 4750 0    60   ~ 0
 PSU_LED
+Text Label 1650 4300 0    60   ~ 0
+PSU_R
 Text Label 1200 4300 2    60   ~ 0
 ARD_R
-Text Label 1650 4300 0    60   ~ 0
-PSU_R
+$Comp
+L R R32
+U 1 1 595DF587
+P 1200 4100
+F 0 "R32" V 1280 4100 50  0000 C CNN
+F 1 "4.7K" V 1200 4100 50  0000 C CNN
+F 2 "Resistors_SMD:R_0805_HandSoldering" V 1130 4100 50  0001 C CNN
+F 3 "" H 1200 4100 50  0001 C CNN
+	1    1200 4100
+	1    0    0    -1
+$EndComp
+$Comp
+L R R33
+U 1 1 595DF58E
+P 1650 4100
+F 0 "R33" V 1730 4100 50  0000 C CNN
+F 1 "4.7K" V 1650 4100 50  0000 C CNN
+F 2 "Resistors_SMD:R_0805_HandSoldering" V 1580 4100 50  0001 C CNN
+F 3 "" H 1650 4100 50  0001 C CNN
+	1    1650 4100
+	1    0    0    -1
+$EndComp
 $EndSCHEMATC
