File: RLS/RLS.kicad_pcb (KiCad board)
At the start: 2 copper layers, 2 parts

Commit message: PCB has begun
I also realized that I created a duplicate folder now in the GitHub...
Parts:
- removed P1: , 40pinRevised
- removed REF**: Molex_UltraFit_6pin_3.50mm, RLS_CustomFootprints:Molex_UltraFit_6pin_3.50mm
- added C1, C2: 15pF, Capacitors_THT:C_Disc_D3.8mm_W2.6mm_P2.50mm, F.Cu at (135.9, 69.8)
- added C10, C12, C14, C22, C24, C26, C28, C30, C32, C39, C4, C40, C6, C8: 0.1uF, Capacitors_SMD:C_0603_HandSoldering, F.Cu at (135.9, 69.8)
- added C11, C13, C17, C18, C19, C20, C21, C23, C25, C27, C29, C3, C31, C35, C36, C37, C38, C41, C42, C45, C5, C7, C9: 10uF, Capacitors_SMD:CP_Elec_4x5.3, F.Cu at (135.9, 69.8)
- added C15, C16, C33, C34, C43, C44: 1uF, Capacitors_SMD:CP_Elec_4x5.3, F.Cu at (135.9, 69.8)
- added D1: AD_LED, LEDs:LED_0603, F.Cu at (135.9, 69.8)
- added D2: +5V_LED, LEDs:LED_0603, F.Cu at (135.9, 69.8)
- added DB1: BoardID_VIN_Scope_FuncGen_DB_CONN, Pin_Headers:Pin_Header_Straight_2x20_Pitch2.54mm, F.Cu at (152.4, 114.3)
- added DB2: Arduino_DB_CONN, Pin_Headers:Pin_Header_Straight_2x20_Pitch2.54mm, F.Cu at (182.9, 104.1)
- added DB3: Logic_Analyzer1_DB_CONN, Pin_Headers:Pin_Header_Straight_2x20_Pitch2.54mm, F.Cu at (254.0, 71.1)
- added DB4: Logic_Analyzer2_DB_CONN, Pin_Headers:Pin_Header_Straight_2x20_Pitch2.54mm, F.Cu at (168.9, 31.8)
- added F1: 1A, Fuse_Holders_and_Fuses:Fuse_SMD2920, F.Cu at (135.9, 69.8)
- added F2: 1.5A, Fuse_Holders_and_Fuses:Fuse_SMD2920, F.Cu at (135.9, 69.8)
- added F3: 4A, Fuse_Holders_and_Fuses:Fuse_SMD2920, F.Cu at (135.9, 69.8)
- added J1: Velleman_Probe1, Pin_Headers:Pin_Header_Straight_1x03_Pitch2.54mm, F.Cu at (135.9, 69.8)
- added J2: Velleman_Probe2, Pin_Headers:Pin_Header_Straight_1x03_Pitch2.54mm, F.Cu at (135.9, 69.8)
- added J3: Velleman_FuncGen, Pin_Headers:Pin_Header_Straight_1x03_Pitch2.54mm, F.Cu at (135.9, 69.8)
- added J4: Logic_Analyzer1, Pin_Headers:Pin_Header_Straight_2x20_Pitch2.54mm, F.Cu at (218.4, 68.6)
- added J5: Logic_Analyzer2, Pin_Headers:Pin_Header_Straight_2x20_Pitch2.54mm, F.Cu at (194.3, 29.2)
- added J6: ADS1115, Pin_Headers:Pin_Header_Straight_1x10_Pitch2.54mm, F.Cu at (64.8, 119.4)
- added J7: DC_Fan, Pin_Headers:Pin_Header_Straight_1x03_Pitch2.54mm, F.Cu at (135.9, 69.8)
- added PSU1: DIN_5, RLS_CustomFootprints:Molex_2x3_3.5mm, F.Cu at (135.9, 69.8)
- added Q1: BS170, TO_SOT_Packages_SMD:SOT-23, F.Cu at (135.9, 69.8)
- added R1, R10, R19, R2, R22, R3, R30, R31, R32, R33, R4, R5, R6, R7, R8, R9: 4.7K, Resistors_SMD:R_0805_HandSoldering, F.Cu at (135.9, 69.8)
- added R11, R13: 20K, Resistors_SMD:R_1206_HandSoldering, F.Cu at (135.9, 69.8)
- added R12, R14, R15, R16: 10K, Resistors_SMD:R_1206_HandSoldering, F.Cu at (135.9, 69.8)
- added R17, R18: 9M, Resistors_THT:R_Axial_DIN0309_L9.0mm_D3.2mm_P12.70mm_Horizontal, F.Cu at (135.9, 69.8)
- added R20, R21, R23, R24: 1.78K, Resistors_SMD:R_1206_HandSoldering, F.Cu at (135.9, 69.8)
- added R25, R28: 120, Resistors_SMD:R_1206_HandSoldering, F.Cu at (135.9, 69.8)
- added R26, R27: 1K_POT, Potentiometers:Potentiometer_Trimmer_Bourns_3296Y, F.Cu at (135.9, 69.8)
- added R29: 1K, Resistors_SMD:R_1206_HandSoldering, F.Cu at (135.9, 69.8)
- added TH1: 3K_NTC, Resistors_THT:R_Axial_DIN0411_L9.9mm_D3.6mm_P12.70mm_Horizontal, F.Cu at (135.9, 69.8)
- added U10, U11: LT1963, TO_SOT_Packages_THT:TO-220-5_Pentawatt_Multiwatt-5_Vertical_StaggeredType1, F.Cu at (135.9, 69.8)
- added U12: ULN2803A, Housings_DIP:DIP-18_W7.62mm, F.Cu at (38.1, 35.6)
- added U2: LM317T, TO_SOT_Packages_THT:TO-220_Vertical, F.Cu at (135.9, 69.8)
- added U3: LM337T, TO_SOT_Packages_THT:TO-220_Vertical, F.Cu at (135.9, 69.8)
- added U4, U5, U8, U9: AD5293, SMD_Packages:SSOP-14, F.Cu at (135.9, 69.8)
- added U6, U7: LT3015, TO_SOT_Packages_THT:TO-220-5_Pentawatt_Multiwatt-5_Vertical_StaggeredType1, F.Cu at (135.9, 69.8)
Other:
- board outline added: 228.6 x 228.6 mm
- copper layers 2 -> 4
- net class Default: clearance 0.2 -> 0.25
- rule trace_clearance: 0.2 -> 0.25
- rule trace_min: 0.2 -> 0.25
